Commit message: robotiq gripper now compatible with matisse project

File: robotiq_description/urdf/2f_140.ros2_control.xacro (robot description, xacro)
@@ -4,5 +4,5 @@
         name
         prefix
-        sim_gazebo:=false
+        sim_ignition:=false
         sim_isaac:=false
         isaac_joint_commands:=/isaac_joint_commands
@@ -15,81 +15,167 @@
         gripper_max_speed:=0.250
         gripper_max_force:=125.0
-        gripper_closed_position:=0.695">
-        <ros2_control name="${name}" type="system">
-            <!-- Plugins -->
-            <hardware>
-                <xacro:if value="${sim_isaac}">
-                    <plugin>topic_based_ros2_control/TopicBasedSystem</plugin>
-                    <param name="joint_commands_topic">${isaac_joint_commands}</param>
-                    <param name="joint_states_topic">${isaac_joint_states}</param>
+        gripper_closed_position:=0.695
+        mounted_on_ur:=false">
+        <xacro:unless value="${mounted_on_ur}">
+            <ros2_control name="${name}" type="system">
+                <!-- Plugins -->
+                <hardware>
+                    <xacro:if value="${sim_isaac}">
+                        <plugin>topic_based_ros2_control/TopicBasedSystem</plugin>
+                        <param name="joint_commands_topic">${isaac_joint_commands}</param>
+                        <param name="joint_states_topic">${isaac_joint_states}</param>
+                    </xacro:if>
+                    <xacro:if value="${sim_ignition}">
+                        <plugin>gz_ros2_control/GazeboSimSystem</plugin>
+                    </xacro:if>
+                    <xacro:if value="${use_fake_hardware}">
+                        <plugin>mock_components/GenericSystem</plugin>
+                        <param name="mock_sensor_commands">${mock_sensor_commands}</param>
+                        <param name="state_following_offset">0.0</param>
+                    </xacro:if>
+                    <xacro:unless value="${use_fake_hardware or sim_ignition or sim_isaac}">
+                        <plugin>robotiq_driver/RobotiqGripperHardwareInterface</plugin>
+                        <param name="gripper_closed_position">${gripper_closed_position}</param>
+                        <param name="COM_port">${com_port}</param>
+                        <param name="gripper_speed_multiplier">${gripper_speed_multiplier}</param>
+                        <param name="gripper_force_multiplier">${gripper_force_multiplier}</param>
+                        <param name="gripper_max_speed">${gripper_max_speed}</param>
+                        <param name="gripper_max_force">${gripper_max_force}</param>
+                    </xacro:unless>
+                </hardware>
+                <!-- Joint interfaces -->
+                <!-- With Ignition or Hardware, they handle mimic joints, so we only need this
+                command interface activated -->
+                <joint name="${prefix}finger_joint">
+                    <command_interface name="position" />
+                    <state_interface name="position">
+                        <param name="initial_value">0.01</param>
+                    </state_interface>
+                    <state_interface name="velocity" />
+                </joint>
+                <!-- When simulating we need to include the rest of the gripper joints -->
+                <xacro:if value="${use_fake_hardware or sim_isaac or sim_ignition}">
+                    <joint name="${prefix}left_inner_knuckle_joint">
+                        <param name="mimic">${prefix}finger_joint</param>
+                        <param name="multiplier">-1</param>
+                        <xacro:unless value="${sim_ignition}">
+                            <command_interface name="position" />
+                            <state_interface name="position" />
+                            <state_interface name="velocity" />
+                        </xacro:unless>
+                    </joint>
+                    <joint name="${prefix}left_inner_finger_joint">
+                        <param name="mimic">${prefix}finger_joint</param>
+                        <param name="multiplier">1</param>
+                        <xacro:unless value="${sim_ignition}">
+                            <command_interface name="position" />
+                            <state_interface name="position" />
+                            <state_interface name="velocity" />
+                        </xacro:unless>
+                    </joint>
+                    <joint name="${prefix}right_outer_knuckle_joint">
+                        <param name="mimic">${prefix}finger_joint</param>
+                        <param name="multiplier">-1</param>
+                        <xacro:unless value="${sim_ignition}">
+                            <command_interface name="position" />
+                            <state_interface name="position" />
+                            <state_interface name="velocity" />
+                        </xacro:unless>
+                    </joint>
+                    <joint name="${prefix}right_inner_knuckle_joint">
+                        <param name="mimic">${prefix}finger_joint</param>
+                        <param name="multiplier">-1</param>
+                        <xacro:unless value="${sim_ignition}">
+                            <command_interface name="position" />
+                            <state_interface name="position" />
+                            <state_interface name="velocity" />
+                        </xacro:unless>
+                    </joint>
+                    <joint name="${prefix}right_inner_finger_joint">
+                        <param name="mimic">${prefix}finger_joint</param>
+                        <param name="multiplier">1</param>
+                        <xacro:unless value="${sim_ignition}">
+                            <command_interface name="position" />
+                            <state_interface name="position" />
+                            <state_interface name="velocity" />
+                        </xacro:unless>
+                    </joint>
                 </xacro:if>
-                <xacro:if value="${sim_gazebo}">
-                    <plugin>gz_ros2_control/GazeboSimSystem</plugin>
-                </xacro:if>
-                <xacro:if value="${use_fake_hardware}">
-                    <plugin>mock_components/GenericSystem</plugin>
-                    <param name="mock_sensor_commands">${mock_sensor_commands}</param>
-                    <param name="state_following_offset">0.0</param>
-                </xacro:if>
-                <xacro:unless value="${use_fake_hardware or sim_gazebo or sim_isaac}">
-                    <plugin>robotiq_driver/RobotiqGripperHardwareInterface</plugin>
-                    <param name="gripper_closed_position">${gripper_closed_position}</param>
-                    <param name="COM_port">${com_port}</param>
-                    <param name="gripper_speed_multiplier">${gripper_speed_multiplier}</param>
-                    <param name="gripper_force_multiplier">${gripper_force_multiplier}</param>
-                    <param name="gripper_max_speed">${gripper_max_speed}</param>
-                    <param name="gripper_max_force">${gripper_max_force}</param>
+                <!-- Only add this with fake hardware mode -->
+                <xacro:unless value="${sim_ignition or sim_isaac}">
+                    <gpio name="reactivate_gripper">
+                        <command_interface name="reactivate_gripper_cmd" />
+                        <command_interface name="reactivate_gripper_response" />
+                    </gpio>
                 </xacro:unless>
-            </hardware>
-            <!-- Joint interfaces -->
-            <!-- With Gazebo or Hardware, they handle mimic joints, so we only need this command interface activated -->
+            </ros2_control>
+        </xacro:unless>
+        <xacro:if value="${mounted_on_ur}">
             <joint name="${prefix}finger_joint">
                 <command_interface name="position" />
                 <state_interface name="position">
-                    <param name="initial_value">${gripper_closed_position}</param>
+                    <param name="initial_value">0.01</param>
                 </state_interface>
-                <state_interface name="velocity"/>
+                <state_interface name="velocity" />
             </joint>
             <!-- When simulating we need to include the rest of the gripper joints -->
-            <xacro:if value="${use_fake_hardware or sim_isaac or sim_gazebo}">
+            <xacro:if value="${use_fake_hardware or sim_isaac or sim_ignition}">
                 <joint name="${prefix}left_inner_knuckle_joint">
-                    <xacro:unless value="${sim_gazebo}">
-                        <state_interface name="position"/>
-                        <state_interface name="velocity"/>
+                    <param name="mimic">${prefix}finger_joint</param>
+                    <param name="multiplier">-1</param>
+                    <xacro:unless value="${sim_ignition}">
+                        <command_interface name="position" />
+                        <state_interface name="position" />
+                        <state_interface name="velocity" />
                     </xacro:unless>
                 </joint>
                 <joint name="${prefix}left_inner_finger_joint">
-                    <xacro:unless value="${sim_gazebo}">
-                        <state_interface name="position"/>
-                        <state_interface name="velocity"/>
+                    <param name="mimic">${prefix}finger_joint</param>
+                    <param name="multiplier">1</param>
+                    <xacro:unless value="${sim_ignition}">
+                        <command_interface name="position" />
+                        <state_interface name="position" />
+                        <state_interface name="velocity" />
                     </xacro:unless>
                 </joint>
                 <joint name="${prefix}right_outer_knuckle_joint">
-                    <xacro:unless value="${sim_gazebo}">
-                        <state_interface name="position"/>
-                        <state_interface name="velocity"/>
+                    <param name="mimic">${prefix}finger_joint</param>
+                    <param name="multiplier">-1</param>
+                    <xacro:unless value="${sim_ignition}">
+                        <command_interface name="position" />
+                        <state_interface name="position" />
+                        <state_interface name="velocity" />
                     </xacro:unless>
                 </joint>
                 <joint name="${prefix}right_inner_knuckle_joint">
-                    <xacro:unless value="${sim_gazebo}">
-                        <state_interface name="position"/>
-                        <state_interface name="velocity"/>
+                    <param name="mimic">${prefix}finger_joint</param>
+                    <param name="multiplier">-1</param>
+                    <xacro:unless value="${sim_ignition}">
+                        <command_interface name="position" />
+                        <state_interface name="position" />
+                        <state_interface name="velocity" />
                     </xacro:unless>
                 </joint>
                 <joint name="${prefix}right_inner_finger_joint">
-                    <xacro:unless value="${sim_gazebo}">
-                        <state_interface name="position"/>
-                        <state_interface name="velocity"/>
+                    <param name="mimic">${prefix}finger_joint</param>
+                    <param name="multiplier">1</param>
+                    <xacro:unless value="${sim_ignition}">
+                        <command_interface name="position" />
+                        <state_interface name="position" />
+                        <state_interface name="velocity" />
                     </xacro:unless>
                 </joint>
             </xacro:if>
-            <!-- Only add this with fake hardware mode -->
-            <xacro:unless value="${sim_gazebo or sim_isaac}">
-                <gpio name="reactivate_gripper">
-                    <command_interface name="reactivate_gripper_cmd" />
-                    <command_interface name="reactivate_gripper_response" />
-                </gpio>
-            </xacro:unless>
-        </ros2_control>
+        </xacro:if>
+        <xacro:unless value="${mounted_on_ur}">
+            <xacro:if value="${sim_ignition}">
+                <gazebo>
+                    <plugin filename="gz_ros2_control-system"
+                        name="gz_ros2_control::GazeboSimROS2ControlPlugin">
+                        <parameters>/root/ros_workspaces/ros2/matisse_ws/install/robotiq_description/share/robotiq_description/config/robotiq_controllers.yaml</parameters>
+                    </plugin>
+                </gazebo>
+            </xacro:if>
+        </xacro:unless>
     </xacro:macro>
 </robot>

File: robotiq_description/urdf/robotiq_2f_140.xacro (robot description, xacro)
@@ -17,5 +17,5 @@
         <origin xyz="0 0 0" rpy="0 0 0" />
         <geometry>
-          <mesh filename="package://robotiq_description/meshes/visual/2f_140/robotiq_2f_${stroke}_outer_knuckle.stl" />
+          <mesh filename="file://$(find robotiq_description)/meshes/visual/2f_140/robotiq_2f_${stroke}_outer_knuckle.stl" />
         </geometry>
         <material name="">
@@ -26,5 +26,5 @@
         <origin xyz="0 0 0" rpy="0 0 0" />
         <geometry>
-          <mesh filename="package://robotiq_description/meshes/collision/2f_140/robotiq_2f_${stroke}_outer_knuckle.stl" />
+          <mesh filename="file://$(find robotiq_description)/meshes/collision/2f_140/robotiq_2f_${stroke}_outer_knuckle.stl" />
         </geometry>
       </collision>
@@ -47,5 +47,5 @@
         <origin xyz="0 0 0" rpy="0 0 0" />
         <geometry>
-          <mesh filename="package://robotiq_description/meshes/visual/2f_140/robotiq_2f_${stroke}_outer_finger.stl" />
+          <mesh filename="file://$(find robotiq_description)/meshes/visual/2f_140/robotiq_2f_${stroke}_outer_finger.stl" />
         </geometry>
         <material name="">
@@ -56,5 +56,5 @@
         <origin xyz="0 0 0" rpy="0 0 0" />
         <geometry>
-          <mesh filename="package://robotiq_description/meshes/collision/2f_140/robotiq_2f_${stroke}_outer_finger.stl" />
+          <mesh filename="file://$(find robotiq_description)/meshes/collision/2f_140/robotiq_2f_${stroke}_outer_finger.stl" />
         </geometry>
       </collision>
@@ -77,5 +77,5 @@
         <origin xyz="0 0 0" rpy="0 0 0" />
         <geometry>
-          <mesh filename="package://robotiq_description/meshes/visual/2f_140/robotiq_2f_${stroke}_inner_knuckle.stl" />
+          <mesh filename="file://$(find robotiq_description)/meshes/visual/2f_140/robotiq_2f_${stroke}_inner_knuckle.stl" />
         </geometry>
         <material name="">
@@ -83,10 +83,10 @@
         </material>
       </visual>
-      <collision>
+      <!-- <collision>
         <origin xyz="0 0 0" rpy="0 0 0" />
         <geometry>
           <mesh filename="package://robotiq_description/meshes/collision/2f_140/robotiq_2f_${stroke}_inner_knuckle.stl" />
         </geometry>
-      </collision>
+      </collision> -->
     </link>
   </xacro:macro>
@@ -107,5 +107,5 @@
         <origin xyz="0 0 0" rpy="0 0 0" />
         <geometry>
-          <mesh filename="package://robotiq_description/meshes/visual/2f_140/robotiq_2f_${stroke}_inner_finger.stl" />
+          <mesh filename="file://$(find robotiq_description)/meshes/visual/2f_140/robotiq_2f_${stroke}_inner_finger.stl" />
         </geometry>
         <material name="">
@@ -116,5 +116,5 @@
         <origin xyz="0 0 0" rpy="0 0 0" />
         <geometry>
-          <mesh filename="package://robotiq_description/meshes/collision/2f_140/robotiq_2f_${stroke}_inner_finger.stl" />
+          <mesh filename="file://$(find robotiq_description)/meshes/collision/2f_140/robotiq_2f_${stroke}_inner_finger.stl" />
         </geometry>
       </collision>
@@ -150,5 +150,5 @@
       <child link="${prefix}left_outer_knuckle" />
       <axis xyz="-1 0 0" />
-      <limit lower="0" upper="0.7" velocity="2.0" effort="1000" />
+      <limit lower="-0.01" upper="0.71" velocity="2.0" effort="70" />
     </joint>
     <xacro:finger_joints prefix="${prefix}" fingerprefix="left" reflect="1.0"/>
@@ -160,5 +160,6 @@
       <child link="${prefix}right_outer_knuckle" />
       <axis xyz="1 0 0" />
-      <limit lower="-0.725" upper="0.725" velocity="2.0" effort="1000" />
+      <limit lower="-0.725" upper="0.725" velocity="5.0" effort="70" />
+      <dynamics damping="5.0" friction="2.0"/>
     <mimic joint="${prefix}finger_joint" multiplier="-1" offset="0" />
     </joint>
@@ -179,5 +180,6 @@
       <child link="${prefix}${fingerprefix}_inner_knuckle" />
       <axis xyz="1 0 0" />
-      <limit lower="-0.8757" upper="0.8757" velocity="2.0" effort="1000" />
+      <limit lower="-0.8757" upper="0.8757" velocity="5.0" effort="70" />
+      <dynamics damping="5.0" friction="2.0"/>
       <mimic joint="${prefix}finger_joint" multiplier="-1" offset="0" />
     </joint>
@@ -189,5 +191,6 @@
       <child link="${prefix}${fingerprefix}_inner_finger" />
       <axis xyz="1 0 0" />
-      <limit lower="-0.8757" upper="0.8757" velocity="2.0" effort="1000" />
+      <limit lower="-0.8757" upper="0.8757" velocity="5.0" effort="70" />
+      <dynamics damping="5.0" friction="2.0"/>
       <mimic joint="${prefix}finger_joint" multiplier="1" offset="0" />
     </joint>

File: robotiq_description/urdf/robotiq_2f_140_macro.urdf.xacro (robot description, xacro)
@@ -6,5 +6,5 @@
         parent
         *origin
-        sim_gazebo:=false
+        sim_ignition:=false
         sim_isaac:=false
         isaac_joint_commands:=/isaac_joint_commands
@@ -18,24 +18,28 @@
         gripper_max_speed:=0.250
         gripper_max_force:=125.0
-        gripper_closed_position:=0.695">
-        <!-- ros2 control include -->
-        <xacro:include filename="$(find robotiq_description)/urdf/2f_140.ros2_control.xacro" />
-        <!-- if we are simulating or directly communicating with the gripper we need a ros2 control instance -->
-        <xacro:if value="${include_ros2_control}">
-            <xacro:robotiq_gripper_ros2_control
-                name="${name}" prefix="${prefix}"
-                sim_gazebo="${sim_gazebo}"
-                sim_isaac="${sim_isaac}"
-                isaac_joint_commands="${isaac_joint_commands}"
-                isaac_joint_states="${isaac_joint_states}"
-                use_fake_hardware="${use_fake_hardware}"
-                mock_sensor_commands="${mock_sensor_commands}"
-                com_port="${com_port}"
-                gripper_speed_multiplier="${gripper_speed_multiplier}"
-                gripper_force_multiplier="${gripper_force_multiplier}"
-                gripper_max_speed="${gripper_max_speed}"
-                gripper_max_force="${gripper_max_force}"
-                gripper_closed_position="${gripper_closed_position}"/>
-        </xacro:if>
+        gripper_closed_position:=0.695
+        mounted_on_ur:=false">
+        <xacro:unless value="${mounted_on_ur}">
+          <!-- ros2 control include -->
+          <xacro:include filename="$(find robotiq_description)/urdf/2f_140.ros2_control.xacro" />
+          <!-- if we are simulating or directly communicating with the gripper we need a ros2 control instance -->
+          <xacro:if value="${include_ros2_control}">
+              <xacro:robotiq_gripper_ros2_control
+                  name="${name}" prefix="${prefix}"
+                  sim_ignition="${sim_ignition}"
+                  sim_isaac="${sim_isaac}"
+                  isaac_joint_commands="${isaac_joint_commands}"
+                  isaac_joint_states="${isaac_joint_states}"
+                  use_fake_hardware="${use_fake_hardware}"
+                  mock_sensor_commands="${mock_sensor_commands}"
+                  com_port="${com_port}"
+                  gripper_speed_multiplier="${gripper_speed_multiplier}"
+                  gripper_force_multiplier="${gripper_force_multiplier}"
+                  gripper_max_speed="${gripper_max_speed}"
+                  gripper_max_force="${gripper_max_force}"
+                  gripper_closed_position="${gripper_closed_position}"
+                  mounted_on_ur="${mounted_on_ur}"/>
+          </xacro:if>
+        </xacro:unless>
         <!-- this is a temporary link to rotate the 2f-140 gripper to match the 2f-85 -->
         <link name="${prefix}robotiq_base_link"/>
@@ -54,5 +58,5 @@
           <origin xyz="0 0 0" rpy="0 0 0" />
           <geometry>
-            <mesh filename="package://robotiq_description/meshes/visual/2f_140/robotiq_2f_140_base_link.stl" />
+            <mesh filename="file://$(find robotiq_description)/meshes/visual/2f_140/robotiq_2f_140_base_link.stl" />
           </geometry>
           <material name="">
@@ -63,5 +67,5 @@
           <origin xyz="0 0 0" rpy="0 0 0" />
           <geometry>
-            <mesh filename="package://robotiq_description/meshes/collision/2f_140/robotiq_2f_140_base_link.stl" />
+            <mesh filename="file://$(find robotiq_description)/meshes/collision/2f_140/robotiq_2f_140_base_link.stl" />
           </geometry>
         </collision>
